File: kicad/BalthazarKeyboard3-keycaps.kicad_pcb (KiCad board)
At the start: 2 copper layers, 290.6 x 127 mm, 195 parts, among them J1 USB, J2 USB_B_Micro, J3 PS2 touchpad, J4 ISP, J5 I2C, SW1 ESC, SW10 2, SW11 3, SW12 4, SW13 5, SW14 6, SW15 TAB, SW16 Q, SW17 W, SW18 E, SW19 R, SW2 F1, SW20 T, SW21 Y, SW22 CAPS, SW23 A, SW24 S, SW25 D, SW26 F, SW27 G, SW28 H, SW29 SHIFT, SW3 F2, SW30 NUBS, SW31 Z, SW32 X, SW33 C, SW34 V, SW35 B, SW36 CTRL, SW37 ALT, SW38 GUI, SW39 SPACE, SW4 F3, SW40 SPACE, SW42 LEFT, SW43 DOWN, SW44 RIGHT, SW45 F7, SW46 F8, SW47 F9, SW48 F10, SW49 F11, SW5 F4, SW50 F12, SW51 PRTSCR, SW52 7, SW53 8, SW54 9, SW55 0, SW56 MINUS, SW57 EQUAL, SW58 DELETE, SW59 U, SW6 F5, SW60 I, SW61 O, SW62 P, SW63 LBRC, SW64 RBRC, SW65 BACKSPACE, SW66 J, SW67 K, SW68 L, SW69 SCLN, SW7 F6, SW70 QUOTE, SW71 NUHS, SW72 ENTER, SW73 N, SW74 M, SW75 COMMA, SW76 DOT, SW77 SLASH, SW78 UP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

Commit message: Adding 2 leyer production files
Other:
- rule pad_to_mask_clearance: 0.051 -> 0
Changed lines of the file:
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@@
     (pad_size 1.35 1.35)
     (pad_drill 0.8)
-    (pad_to_mask_clearance 0.051)
-    (solder_mask_min_width 0.25)
+    (pad_to_mask_clearance 0)
     (aux_axis_origin 4.826 172.72)
     (grid_origin 4.826 172.72)
     (visible_elements 7FFFFFFF)
     (pcbplotparams
-      (layerselection 0x010c0_ffffffff)
+      (layerselection 0x010fc_ffffffff)
       (usegerberextensions true)
       (usegerberattributes false)

Commit message: Switching board to 4 layers
Parts:
- moved C6 1.30 mm to (169.1, 71.3)
- moved C8 0.97 mm to (142.4, 62.0)
- moved C7 0.90 mm to (156.1, 77.3), turned to 180 degrees
- moved H3 0.48 mm to (8.66, 135.6)
Routing:
- net GND: track 347.4 -> 39.6 mm, vias 67 -> 691
- net Vcc: track 161.3 -> 152.4 mm
- net col5: track 318.0 -> 326.7 mm
- net col7: track 240.0 -> 248.3 mm
- net row3: track 425.2 -> 432.6 mm
- net col1: track 199.1 -> 192.4 mm
- net col6: track 433.9 -> 438.9 mm
- net col11: track 166.8 -> 171.6 mm
- net col4: track 232.3 -> 236.7 mm
- net col8: track 221.0 -> 225.4 mm
- net col3: track 227.2 -> 230.3 mm
- net row1: track 387.2 -> 390.0 mm
- net row4: track 528.4 -> 531.0 mm
- net row6: track 386.8 -> 384.5 mm
- net row5: track 408.7 -> 410.5 mm
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- added copper zone on In1.Cu, net GND
- added copper zone on In2.Cu, net GND
- removed copper zone on B.Cu, net GND
- removed copper zone on F.Cu, net GND
Other:
- copper layers 2 -> 4

Commit message: Adding fidutials, adding pin descriptions
Parts:
- removed the G*** at (177.3, 54.6)
- removed the REF** at (208.9, 55.2)
- added FID1: Fiducial, Fiducial:Fiducial_0.5mm_Mask1mm, F.Cu at (8.19, 49.9)
- added FID2: Fiducial, Fiducial:Fiducial_0.5mm_Mask1mm, F.Cu at (292.6, 49.9)
- added FID3: Fiducial, Fiducial:Fiducial_0.5mm_Mask1mm, F.Cu at (7.97, 170.4)
- added FID4: Fiducial, Fiducial:Fiducial_0.5mm_Mask1mm, B.Cu at (292.6, 49.9)
- added FID5: Fiducial, Fiducial:Fiducial_0.5mm_Mask1mm, B.Cu at (8.19, 49.9)
- added FID6: Fiducial, Fiducial:Fiducial_0.5mm_Mask1mm, B.Cu at (292.6, 170.5)
Other:
- board text added: "D+"
- board text added: "D-"
- board text added: "GND"
- board text added: "MISO"
- board text added: "MOSI"
- board text added: "PS2c"
- board text added: "PS2d"
- board text added: "RST"
- board text added: "SCK"
- board text added: "SCL"
- board text added: "SDA"
- board text added: "VBUS"
- board text added: "VCC"
- board text removed: "gnd"
- board text removed: "miso"
- board text removed: "mosi"
- board text removed: "reset"
- board text removed: "sck"
- board text removed: "scl"
- board text removed: "sda"
